File: PowerConverter-KiCad/PowerConverter.kicad_sch (KiCad schematic)
At the start: 19 parts, among them Q1 Q_NMOS_GDS, U1 UCC27517AQDBVRQ1, U2 STM32G431RBTx

Commit message: refactor(hardware): Optimize grounding architecture and power stability
 - Fixed AMS1117-3.3 feedback loop to prevent 6.6V overvoltage.
- Implemented 4-wire Kelvin connection (Net-Tie) for precise 10mOhm current sensing.
- Added 10-ohm gate resistor to UCC27517 to prevent MOSFET gate ringing.
- Safely routed UCC27517 IN- pin to GND.
- Isolated HSE (16MHz) crystal ground strictly to digital GND to protect analog signal integrity.
- Ensured C13 is a Tantalum capacitor for LDO stability (Mental note preserved).
Parts:
- added C10, C14, C15, C16, C17: 100nF, symbol Device:C
- added C11, C12, C13: 22uF, symbol Device:C
- added C18, C19, C20, C9: 10uF, symbol Device:C
- added C21: 10nF, symbol Device:C
- added C22, C23: 10p, symbol Device:C
- added D2: LED, symbol Device:LED
- added FB1: 120R, Inductor_SMD:L_0603_1608Metric, symbol Device:FerriteBead
- added L3: 4.7uH, symbol Device:L
- added NT1: NetTie_2, NetTie:NetTie-2_SMD_Pad0.5mm, symbol Device:NetTie_2
- added R6: 10, symbol Device:R_US
- added R7: 100k, symbol Device:R_US
- added R8: 1.5k, symbol Device:R_US
- added U3: AP63205WU, Package_TO_SOT_SMD:TSOT-23-6, symbol Regulator_Switching:AP63205WU
- added U4: AMS1117-3.3, Package_TO_SOT_SMD:SOT-223-3_TabPin2, symbol Regulator_Linear:AMS1117-3.3
- added Y1: 16MHz, Crystal:Crystal_SMD_3225-4Pin_3.2x2.5mm, symbol Device:Crystal_GND24
Connections:
- net +12V: now also C9.1, U3.2 (EN), U3.3 (IN)
- net GNDA: now also U2.27 (VSSA), C19.2, C21.2, NT1.2; no longer C1.2, C3.2, C4.2, C5.2, C6.2, L2.2, R3.2, U1.2 (GND), U1.4 (IN-)
- net Gate: now also R6.2, R7.2; no longer U1.5 (OUT)
- net +3.3V: now reaches U2.1 (VBAT)
- net +3.3V: now also U2.16 (VDD), U2.32 (VDD), U2.48 (VDD), U2.64 (VDD), C13.1, C14.1, C15.1, C16.1, C17.1, C18.1, C20.1, D2.2 (A), FB1.2, U4.2 (VO)
- net GND: now reaches U2.15 (VSS)
- net GND: now also C1.2, C3.2, C4.2, C5.2, C6.2, L2.2, R3.2, U1.2 (GND), U1.4 (IN-), U2.31 (VSS), U2.47 (VSS), U2.63 (VSS), C11.2, C12.2, C13.2, C14.2, C15.2, C16.2, C17.2, C18.2, C20.2, C22.2, C23.2, C9.2, NT1.1, R7.1, R8.1, U3.4 (GND), U4.1 (GND), Y1.2 (G), Y1.4 (G)
- net +3.3VA: now reaches U2.29 (VDDA)
- net +3.3VA: now also C19.1, C21.1, FB1.1
- net HSE_IN: now reaches U2.5 (PF0)
- net HSE_IN: now also C22.1, Y1.1
- net HSE_OUT: now reaches U2.6 (PF1)
- net HSE_OUT: now also C23.1, Y1.3
- new net: C10.1, U3.5 (SW)
- new net: C10.2, L3.1, U3.6 (BST)
- new net: D2.1 (K), R8.2
- new net: R6.1, U1.5 (OUT)
- new net +5V: C11.1, C12.1, L3.2, U3.1 (FB), U4.3 (VI)
Other:
- note added: "***NetTie ı stm in altından birleştircez"
- note added: "Bu iki toprağı (GND ve GNDA) şemada "Net Tie" adı verilen özel bir sembolle tek bir noktada birleştireceğiz. Nerede birleşmeli? Tam olarak R3 (Şönt) direncinin alt bacağında!"
- note added: "Fedai Notu: Şemayı bitirirken LDO çıkışındaki C13 hala sarı tantal kondansatör, değil mi abi?"

Commit message: refactor: STM32G431 işlemci pin eşleşmeleri ve sinyal bütünlüğü iyileştirmeleri
Bu güncelleme ile donanım mimarisi endüstriyel standartlara getirilmiştir:

- Kristal (HSE) pinleri, G431 mimarisine uygun olarak PF0/PF1 bacaklarına taşındı.
- NRST hattı PG10 (Pin 7) üzerine 100nF filtre ile tanımlandı; sistem kararlılığı artırıldı.
- BOOT0 (PB8) pini 10k pull-down direnci ile mühürlenerek kararsız çalışma modları engellendi.
- ADC hassasiyeti için VREF+ ve VDDA filtreleme katları revize edildi.
- Güç katı (5A SEPIC) toprak dönüşleri, analog bölgeden (GNDA) izole edilerek sistem gürültüsü minimize edildi.
- LDO kararlılığı için C13 kapasitör tipi Tantal olarak belirlendi.
Parts:
- added C24, C25: 100nF, symbol Device:C
- added R9: 10k, symbol Device:R_US
Connections:
- net +3.3VA: now also C25.1
- net GND: now also C24.1, R9.1
- net at U2.28 (VREF+): now also C25.2
- net SWDIO: now reaches U2.49 (PA13)
- net SWDCLK: now reaches U2.50 (PA14)
- net at U2.61 (PB8): now also R9.2
- net at U2.7 (PG10): now also C24.2
Other:
- moved on the sheet: C1, C10, C11, C12, C13, C14, C15, C16, C17, C18, C19, C2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
